Commit message: 2D additions and 3D initial setup

File: src/CrazyS/rotors_description/urdf/haptic_drone_with_structure.xacro (robot description, xacro)
@@ -128,5 +128,5 @@
   </xacro:vertical_rotor>
   <!-- Include the force sensor -->
-  <xacro:include filename="$(find rotors_description)/urdf/nano17.urdf.xacro" />
+  <xacro:include filename="$(find rotors_description)/urdf/nano17_structure.urdf.xacro" />
   <!-- Include the cage -->
   <xacro:include filename="$(find rotors_description)/urdf/cage.urdf" />

File: src/CrazyS/rotors_description/urdf/nano17.urdf.xacro (robot description, xacro)
@@ -3,5 +3,5 @@
 	<!-- Include the force-torque-sensor model -->
 	<xacro:include filename="$(find rotors_description)/urdf/ft_sensor.urdf.xacro"/>
-	<xacro:ft_sensor parent="haptic_drone_with_structure/base_link" name="FT_sensor" type="nano17">
+	<xacro:ft_sensor parent="haptic_drone/base_link" name="FT_sensor" type="nano17">
 		<origin xyz="0 0 -0.02" rpy="0 0 0"/>
 	</xacro:ft_sensor>

File: src/planar_structure/urdf/obstacle_link_joint.xacro (robot description, xacro)
@@ -63,3 +63,7 @@
     </link>
   </xacro:macro>
+  <xacro:macro name="m_link_virtual" params="name">
+    <link name="${name}">
+    </link>
+  </xacro:macro>
 </robot>
