Commit message: Cylindrical obstacles added

File: src/planar_structure/urdf/obstacle_link_joint.xacro (robot description, xacro)
@@ -42,4 +42,25 @@
     </link>
   </xacro:macro>
+  <xacro:macro name="m_link_cyl" params="name origin_xyz origin_rpy radius length mass ixx ixy ixz iyy iyz izz">
+    <link name="${name}">
+      <inertial>
+        <mass value="${mass}" />
+        <origin rpy="${origin_rpy}" xyz="${origin_xyz}" />
+        <inertia ixx="${ixx}" ixy="${ixy}" ixz="${ixz}" iyy="${iyy}" iyz="${iyz}" izz="${izz}" />
+      </inertial>
+      <collision>
+        <origin rpy="${origin_rpy}" xyz="${origin_xyz}" />
+        <geometry>
+	  <cylinder radius="${radius}" length="${length}" />
+        </geometry>
+      </collision>
+      <visual>
+        <origin rpy="${origin_rpy}" xyz="${origin_xyz}" />
+        <geometry>
+          <cylinder radius="${radius}" length="${length}" />
+        </geometry>
+      </visual>
+    </link>
+  </xacro:macro>
   <xacro:macro name="m_link_mesh" params="name origin_xyz origin_rpy meshfile meshscale mass ixx ixy ixz iyy iyz izz">
     <link name="${name}">

File: src/planar_structure/urdf/vertical_obstacle.xacro (robot description, xacro)
@@ -38,5 +38,5 @@
     <plugin name="joint_spring" filename="libjoint_torsional_spring_plugin.so">
       <kx>5</kx>
-      <set_point>-0.01</set_point>
+      <set_point>-0.02</set_point>
       <joint>branch_joint</joint>
     </plugin>

File: src/planar_structure/urdf/vertical_obstacle_closer.xacro (robot description, xacro)
@@ -38,5 +38,5 @@
   <!-- Macro for Torsional Joint Spring Plugin -->
   <gazebo>
-    <plugin name="joint_spring" filename="libgazebo_joint_torsional_spring.so">
+    <plugin name="joint_spring" filename="libjoint_torsional_spring_plugin.so">
       <kx>100</kx>
       <set_point>0.01</set_point>

File: src/planar_structure/urdf/vertical_obstacle_higher.xacro (robot description, xacro)
@@ -38,7 +38,7 @@
   <!-- Macro for Torsional Joint Spring Plugin -->
   <gazebo>
-    <plugin name="joint_spring" filename="libgazebo_joint_torsional_spring.so">
-      <kx>50</kx>
-      <set_point>0.3</set_point>
+    <plugin name="joint_spring" filename="libjoint_torsional_spring_plugin.so">
+      <kx>5</kx>
+      <set_point>-0.02</set_point>
       <joint>${link_00_name}_${link_01_name}_joint</joint>
     </plugin>
